File: Shield_Emergent_4/Shield_Emergent_4.kicad_pcb (KiCad board)
At the start: 4 copper layers, 23.6 x 33.4 mm, 29 parts, among them J1 USB3_B_Micro, J2 Conn_01x04_Socket, J3 USB3_B_Micro, J4 Conn_01x05, J5 Conn_01x02_Socket, J6 Conn_01x02_Socket, J7 Conn_01x05, J8 Conn_01x10, U3 SP3012-06UTG, U4 SP3012-06UTG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

Commit message: v0.3 LF circuits were routed
Parts:
- D1: moved to F.Cu
- moved C2 6.50 mm to (23.8, 11.9), turned to 180 degrees
- moved U1 5.39 mm to (23.8, 8.70)
- moved R6 4.47 mm to (21.2, 8.90)
- moved R4 3.10 mm to (20.2, 7.10)
- moved D1 2.95 mm to (24.4, 3.65), turned to 0 degrees
- moved J5 0.51 mm to (24.1, 14.8), turned to 90 degrees
Connections:
- J1 pad 2: D- -> 1_D-
- J1 pad 3: D+ -> 1_D+
- U3 pad 6: D+ -> 1_D+
- U3 pad 7: D- -> 1_D-
- U3 pad 8: D- -> 1_D-
- U3 pad 9: D+ -> 1_D+
Routing:
- net VBUS: track 88.8 -> 104.4 mm, vias 20 -> 21
- net D+: track 23.8 -> 13.3 mm
- net 1_D+: track 0.00 -> 10.5 mm
- net D-: track 23.4 -> 15.1 mm
- net 1_D-: track 0.00 -> 8.25 mm
- net EN1: track 5.95 -> 12.2 mm
- net nFLT1: track 6.93 -> 12.0 mm, vias 0 -> 1
- net VOUT1: track 21.9 -> 19.2 mm, vias 7 -> 9
- net Net-(U1-ILIM): track 1.90 -> 3.75 mm
- net GND: vias 140 -> 139
