File: Shield_Emergent_4/Shield_Emergent_4.kicad_pcb (KiCad board)
At the start: 4 copper layers, 23.6 x 33.4 mm, 29 parts, among them J1 USB3_B_Micro, J2 Conn_01x04_Socket, J3 USB3_B_Micro, J4 Conn_01x05, J5 Conn_01x02_Socket, J6 Conn_01x02_Socket, J7 Conn_01x05, J8 Conn_01x10, U3 SP3012-06UTG, U4 SP3012-06UTG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

Commit message: v0.4 Seems 2B ready
Parts:
- moved C2 0.25 mm to (22.2, 18.2)
Routing:
- net VBUS: track 88.8 -> 99.4 mm
- net D+: track 23.8 -> 27.6 mm
- net K7: track 8.91 -> 11.2 mm
- net K2: track 7.84 -> 9.36 mm
- net K1: track 6.92 -> 8.02 mm
- net D-: track 23.4 -> 24.2 mm
- net K3: track 6.36 -> 7.07 mm
- net K5: track 6.73 -> 7.29 mm
- net GND: vias 140 -> 146

Commit message: v0.5 modified and ordered
Connections:
- J1 pad 2: D- -> 1_D-
- J1 pad 3: D+ -> 1_D+
- U3 pad 6: D+ -> 1_D+
- U3 pad 7: D- -> 1_D-
- U3 pad 8: D- -> 1_D-
- U3 pad 9: D+ -> 1_D+
Routing:
- net D+: track 27.6 -> 16.1 mm
- net 1_D+: track 0.00 -> 10.5 mm
- net D-: track 24.2 -> 15.9 mm
- net 1_D-: track 0.00 -> 8.25 mm
- net VOUT1: track 21.9 -> 28.9 mm, vias 7 -> 10
- net VOUT2: track 33.8 -> 39.1 mm, vias 10 -> 15
- net VBUS: track 99.4 -> 102.8 mm, vias 20 -> 23

Commit message: v0.6 new geometry
Parts:
- added R10: 0, Resistor_SMD:R_0201_0603Metric_Pad0.64x0.40mm_HandSolder, F.Cu at (59.6, 53.5)
- added R11: 0, Resistor_SMD:R_0201_0603Metric_Pad0.64x0.40mm_HandSolder, F.Cu at (59.6, 55.2)
- added R12: 0, Resistor_SMD:R_0201_0603Metric_Pad0.64x0.40mm_HandSolder, F.Cu at (59.6, 57.0)
- added R9: 0, Resistor_SMD:R_0201_0603Metric_Pad0.64x0.40mm_HandSolder, F.Cu at (59.6, 51.8)
- J1, J3: value USB3_B_Micro -> TF31-18S-0.5SH_800_; footprint USB_Conns:MU3MS04 -> my8lib:HRS_TF31-18S-0.5SH_800_; moved to F.Cu
- J8: value Conn_01x10 -> Conn_02x05_Odd_Even; footprint myLib8:50A-10LB -> Connector_PinHeader_1.27mm:PinHeader_2x05_P1.27mm_Vertical
- U5: moved to F.Cu
- moved U5 76.8 mm to (73.9, 40.0), turned to 180 degrees
- moved J7 76.1 mm to (71.8, 34.5), turned to -90 degrees
- moved J4 76.0 mm to (71.7, 42.0), turned to -90 degrees
- moved U6 72.6 mm to (73.7, 37.0), turned to 180 degrees
- moved C1 71.5 mm to (85.2, 41.5)
- moved C2 71.5 mm to (85.5, 51.7)
- moved C4 71.5 mm to (70.2, 56.5)
- moved D2 71.5 mm to (71.0, 58.5)
- moved R1 71.5 mm to (74.9, 43.8)
- moved R2 71.5 mm to (80.7, 43.6)
- moved R3 71.5 mm to (76.8, 55.7)
- moved R5 71.5 mm to (81.0, 53.2)
- moved R6 71.5 mm to (82.0, 46.1)
- moved R7 71.5 mm to (77.4, 65.9)
- moved U1 71.5 mm to (84.3, 46.9)
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Connections:
- J1 pad 1: VOUT1 -> GND
- J1 pad 10: RX1+ -> unconnected-(J1-Pad10)
- J1 pad 2: 1_D- -> RX1+
- J1 pad 3: 1_D+ -> GND
- J1 pad 4: unconnected-(J1-ID-Pad4) -> RX1-
- J1 pad 6: TX1- -> TX1+
- J1 pad 7: TX1+ -> GND
- J1 pad 8: GND -> TX1-
- J1 pad 9: RX1- -> GND
- J3 pad 1: VOUT2 -> GND
- J3 pad 10: RX2+ -> unconnected-(J3-Pad10)
- J3 pad 2: 2_D- -> RX2+
- J3 pad 3: 2_D+ -> GND
- J3 pad 4: unconnected-(J3-ID-Pad4) -> RX2-
- J3 pad 7: TX2- -> GND
- J3 pad 8: GND -> TX2-
- J3 pad 9: RX2- -> GND
- U5 pad 11: K4 -> K7
- U5 pad 12: K3 -> K5
- U5 pad 13: K2 -> K3
- U5 pad 2: K2 -> K3
- U5 pad 3: K3 -> K5
- U5 pad 4: K4 -> K7
- U5 pad 6: K5 -> K9
- U5 pad 7: K6 -> unconnected-(U5-Pad7)
- U5 pad 8: K6 -> unconnected-(U5-Pad8)
- U5 pad 9: K5 -> K9
- U6 pad 1: K9 -> K2
- U6 pad 11: unconnected-(U6-Pad11) -> K8
- U6 pad 12: K7 -> K6
- U6 pad 13: K8 -> K4
- U6 pad 14: K9 -> K2
- U6 pad 2: K8 -> K4
- U6 pad 3: K7 -> K6
- U6 pad 4: unconnected-(U6-Pad4) -> K8
Routing:
- net K3: track 7.07 -> 14.4 mm
- net K5: track 7.29 -> 14.3 mm
- net K8: track 7.84 -> 13.6 mm
- net K1: track 8.02 -> 13.7 mm
- net K4: track 8.77 -> 13.9 mm
- net K6: track 8.06 -> 13.2 mm
- net K2: track 9.36 -> 13.6 mm
- net K9: track 10.2 -> 14.1 mm
- net K7: track 11.2 -> 13.6 mm
- net GND: vias 146 -> 142
Other:
- board size 23.6 x 33.4 mm -> 89 x 67.1 mm

Commit message: v0.7 predecomposition was completed
Parts:
- C2, C3: footprint Capacitor_SMD:C_0603_1608Metric_Pad1.08x0.95mm_HandSolder -> Capacitor_SMD:C_0402_1005Metric_Pad0.74x0.62mm_HandSolder; moved to F.Cu
- D1, D2, U1, U2: moved to F.Cu
- J5: footprint Connector_PinSocket_2.00mm:PinSocket_1x02_P2.00mm_Vertical -> Connector_PinHeader_1.27mm:PinHeader_1x02_P1.27mm_Vertical; moved to F.Cu
- J6: footprint Connector_PinSocket_2.54mm:PinSocket_1x02_P2.54mm_Vertical -> Connector_PinHeader_1.27mm:PinHeader_1x02_P1.27mm_Vertical
- R1, U5: moved to B.Cu
- R4, R8: footprint Resistor_SMD:R_0603_1608Metric_Pad0.98x0.95mm_HandSolder -> Resistor_SMD:R_0402_1005Metric_Pad0.72x0.64mm_HandSolder; moved to F.Cu
- R6: footprint Resistor_SMD:R_0402_1005Metric -> Resistor_SMD:R_0402_1005Metric_Pad0.72x0.64mm_HandSolder; moved to F.Cu
- R7: footprint Resistor_SMD:R_0402_1005Metric -> Resistor_SMD:R_0402_1005Metric_Pad0.72x0.64mm_HandSolder
- moved C2 94.6 mm to (1.00, 9.00)
- moved C1 88.8 mm to (4.80, 3.80), turned to 180 degrees
- moved U1 88.6 mm to (4.00, 9.40), turned to 0 degrees
- moved J5 88.1 mm to (8.00, 11.2), turned to 180 degrees
- moved J6 85.4 mm to (11.1, 25.2)
- moved R6 85.2 mm to (4.00, 11.8), turned to 180 degrees
- moved R4 83.8 mm to (7.60, 8.20), turned to 0 degrees
- moved D1 80.9 mm to (13.4, 7.80), turned to 0 degrees
- moved U4 79.1 mm to (10.7, 19.0), turned to 0 degrees
- moved J3 78.4 mm to (2.81, 19.8)
- moved R7 74.3 mm to (11.2, 32.2), turned to 0 degrees
- moved R3 73.6 mm to (15.1, 15.6), turned to 0 degrees
- moved R12 73.4 mm to (1.80, 11.8), turned to 180 degrees
- moved D2 72.5 mm to (7.80, 23.0), turned to 90 degrees
- moved C3 72.0 mm to (11.2, 31.0), turned to 180 degrees
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Connections:
- J3 pad 6: TX2+ -> TX2-
- J3 pad 8: TX2- -> TX2+
Routing:
- net VBUS: track 102.8 -> 0.00 mm, vias 23 -> 0
- net VOUT2: track 39.1 -> 0.21 mm, vias 15 -> 0
- net VOUT1: track 28.9 -> 0.00 mm, vias 10 -> 0
- net nFLT2: track 18.6 -> 0.00 mm, vias 1 -> 0
- net D+: track 16.1 -> 0.70 mm
- net D-: track 15.9 -> 0.70 mm, vias 2 -> 0
- net EN2: track 15.2 -> 0.00 mm
- net K3: track 14.4 -> 0.00 mm, vias 1 -> 0
- net K5: track 14.3 -> 0.00 mm, vias 1 -> 0
- net K9: track 14.1 -> 0.00 mm, vias 1 -> 0
- net K4: track 13.9 -> 0.00 mm, vias 1 -> 0
- net K1: track 13.7 -> 0.00 mm, vias 1 -> 0
- net K2: track 13.6 -> 0.00 mm, vias 1 -> 0
- net K7: track 13.6 -> 0.00 mm, vias 1 -> 0
- net K8: track 13.6 -> 0.00 mm, vias 1 -> 0
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- removed copper zone on B.Cu, net GND
- removed copper zone on F.Cu, net GND
- removed copper zone on In1.Cu, net GND
- removed copper zone on In2.Cu, net GND

Commit message: м0,8 reflection was committed
Parts:
- moved C2 25.1 mm to (26.1, 9.00)
- moved R12 23.5 mm to (25.3, 11.8), turned to 0 degrees
- moved R11 22.3 mm to (24.7, 27.6), turned to 0 degrees
- moved J3 21.5 mm to (24.3, 19.8), turned to -90 degrees
- moved J2 21.3 mm to (2.88, 22.8)
- moved R6 19.1 mm to (23.1, 11.8), turned to 0 degrees
- moved U1 19.1 mm to (23.1, 9.40), turned to 180 degrees
- moved R2 17.9 mm to (4.63, 15.6), turned to 0 degrees
- moved R5 17.9 mm to (4.63, 20.4), turned to 0 degrees
- moved C4 17.5 mm to (22.3, 31.8), turned to 0 degrees
- moved R4 11.9 mm to (19.5, 8.20), turned to 180 degrees
- moved D2 11.5 mm to (19.3, 23.0)
- moved R8 11.1 mm to (19.1, 27.2)
- moved J5 11.1 mm to (19.1, 11.2)
- moved X1 10.3 mm to (8.43, 18.0), turned to 180 degrees
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Routing:
- net D-: track 0.70 -> 0.00 mm
- net D+: track 0.70 -> 0.00 mm
