File: Shield_Emergent_4/Shield_Emergent_4.kicad_sch (KiCad schematic)
At the start: 29 parts, among them J1 USB3_B_Micro, J2 Conn_01x04_Socket, J3 USB3_B_Micro, J4 Conn_01x05, J5 Conn_01x02_Socket, J6 Conn_01x02_Socket, J7 Conn_01x05, J8 Conn_01x10, U3 SP3012-06UTG, U4 SP3012-06UTG, U5 SP3012-06UTG, U6 SP3012-06UTG, X1 USB_C_24pins

Commit message: v0.5 modified and ordered
Connections:
- net D+: no longer J1.3 (D+), U3.6, U3.9
- net D-: no longer J1.2 (D-), U3.7, U3.8
- new net 1_D+: J1.3 (D+), U3.6, U3.9
- new net 1_D-: J1.2 (D-), U3.7, U3.8

Commit message: v0.6 new geometry
Parts:
- removed J1, J3: USB3_B_Micro, USB_Conns:MU3MS04, symbol Connector:USB3_B_Micro
- removed J8: Conn_01x10, myLib8:50A-10LB, symbol Vedrofara:Conn_01x10
- added J1, J3: TF31-18S-0.5SH_800_, my8lib:HRS_TF31-18S-0.5SH_800_, symbol my8lib:TF31-18S-0.5SH_800_
- added J8: Conn_02x05_Odd_Even, Connector_PinHeader_1.27mm:PinHeader_2x05_P1.27mm_Vertical, symbol Connector_Generic:Conn_02x05_Odd_Even
- added R10, R11, R12, R9: 0, Resistor_SMD:R_0201_0603Metric_Pad0.64x0.40mm_HandSolder, symbol Device:R
Connections:
- net 1_D+: now also J1.12
- net 1_D-: now also J1.14
- net 2_D+: now also J3.12
- net 2_D-: now also J3.14
- net GND: now also J1.1, J1.11, J1.13, J1.15, J1.16, J1.3, J1.5, J1.7, J1.9, J3.1, J3.11, J3.13, J3.15, J3.16, J3.3, J3.5, J3.7, J3.9, J8.10 (Pin_10), R10.2, R11.2, R12.2, R9.2
- net K1: now also J8.1 (Pin_1)
- net K2: now also U6.1, U6.14, J8.2 (Pin_2); no longer U5.13, U5.2
- net K3: now also U5.13, U5.2, J8.3 (Pin_3); no longer U5.12, U5.3
- net K4: now also U6.13, U6.2, J8.4 (Pin_4); no longer U5.11, U5.4
- net K5: now also U5.12, U5.3, J8.5 (Pin_5); no longer U5.6, U5.9
- net K6: now also U6.12, U6.3, J8.6 (Pin_6); no longer U5.7, U5.8
- net K7: now also U5.11, U5.4, J8.7 (Pin_7); no longer U6.12, U6.3
- net K8: now also U6.11, U6.4, J8.8 (Pin_8); no longer U6.13, U6.2
- net K9: now also U5.6, U5.9, J8.9 (Pin_9); no longer U6.1, U6.14
- net RX1+: now also J1.2
- net RX1-: now also J1.4
- net RX2+: now also J3.2
- net RX2-: now also J3.4
- net TX1+: now also J1.6
- net TX1-: now also J1.8
- net TX2+: now also J3.6
- net TX2-: now also J3.8
- net VOUT1: now also J1.17, J1.18
- net VOUT2: now also J3.17, J3.18
- new net: J1.S1, R9.1
- new net: J1.S2, R10.1
- new net: J3.S1, R11.1
- new net: J3.S2, R12.1
Other:
- moved on the sheet: D1, D2, J4, J7

Commit message: v0.7 predecomposition was completed
Parts:
- C2, C3: footprint Capacitor_SMD:C_0603_1608Metric_Pad1.08x0.95mm_HandSolder -> Capacitor_SMD:C_0402_1005Metric_Pad0.74x0.62mm_HandSolder
- J5: footprint Connector_PinSocket_2.00mm:PinSocket_1x02_P2.00mm_Vertical -> Connector_PinHeader_1.27mm:PinHeader_1x02_P1.27mm_Vertical
- J6: footprint Connector_PinSocket_2.54mm:PinSocket_1x02_P2.54mm_Vertical -> Connector_PinHeader_1.27mm:PinHeader_1x02_P1.27mm_Vertical
- R4, R8: footprint Resistor_SMD:R_0603_1608Metric_Pad0.98x0.95mm_HandSolder -> Resistor_SMD:R_0402_1005Metric_Pad0.72x0.64mm_HandSolder
- R6, R7: footprint Resistor_SMD:R_0402_1005Metric -> Resistor_SMD:R_0402_1005Metric_Pad0.72x0.64mm_HandSolder
Connections:
- net TX2+: now also J3.8; no longer J3.6
- net TX2-: now also J3.6; no longer J3.8
Changed lines of the file:
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@@
 		)
 	)
+	(global_label "TX2-"
+		(shape input)
+		(at 246.38 96.52 180)
+		(fields_autoplaced yes)
+		(effects
+			(font
+				(size 1.27 1.27)
+			)
+			(justify right)
+		)
+		(property "Intersheetrefs" "${INTERSHEET_REFS}"
+			(at 238.4358 96.52 0)
+			(effects
+				(font
+					(size 1.27 1.27)
+				)
+				(justify right)
+				(hide yes)
+			)
+		)
+	)
 	(global_label "TX1+"
 		(shape input)
@@
 		)
 	)
-	(global_label "TX2-"
-		(shape input)
-		(at 246.38 101.6 180)
-		(fields_autoplaced yes)
-		(effects
-			(font
-				(size 1.27 1.27)
-			)
-			(justify right)
-		)
-		(property "Intersheetrefs" "${INTERSHEET_REFS}"
-			(at 238.4358 101.6 0)
-			(effects
-				(font
-					(size 1.27 1.27)
-				)
-				(justify right)
-				(hide yes)
-			)
-		)
-	)
 	(global_label "K4"
 		(shape input)
@@
 		)
 	)
-	(global_label "TX2+"
-		(shape input)
-		(at 246.38 96.52 180)
-		(fields_autoplaced yes)
-		(effects
-			(font
-				(size 1.27 1.27)
-			)
-			(justify right)
-		)
-		(property "Intersheetrefs" "${INTERSHEET_REFS}"
-			(at 238.4358 96.52 0)
-			(effects
-				(font
-					(size 1.27 1.27)
-				)
-				(justify right)
-				(hide yes)
-			)
-		)
-	)
 	(global_label "nFLT2"
 		(shape input)
@@
 		)
 	)
+	(global_label "TX2+"
+		(shape input)
+		(at 246.38 101.6 180)
+		(fields_autoplaced yes)
+		(effects
+			(font
+				(size 1.27 1.27)
+			)
+			(justify right)
+		)
+		(property "Intersheetrefs" "${INTERSHEET_REFS}"
+			(at 238.4358 101.6 0)
+			(effects
+				(font
+					(size 1.27 1.27)
+				)
+				(justify right)
+				(hide yes)
+			)
+		)
+	)
 	(global_label "TX2-"
 		(shape input)
@@
 			)
 		)
-		(property "Footprint" "Resistor_SMD:R_0603_1608Metric_Pad0.98x0.95mm_HandSolder"
+		(property "Footprint" "Resistor_SMD:R_0402_1005Metric_Pad0.72x0.64mm_HandSolder"
 			(at 145.542 72.39 90)
 			(effects
@@
 			)
 		)
-		(property "Footprint" "Resistor_SMD:R_0402_1005Metric"
+		(property "Footprint" "Resistor_SMD:R_0402_1005Metric_Pad0.72x0.64mm_HandSolder"
 			(at 113.03 61.468 90)
 			(effects
@@
 			)
 		)
-		(property "Footprint" "Resistor_SMD:R_0603_1608Metric_Pad0.98x0.95mm_HandSolder"
+		(property "Footprint" "Resistor_SMD:R_0402_1005Metric_Pad0.72x0.64mm_HandSolder"
 			(at 146.812 36.83 90)
 			(effects
@@
 			)
 		)
-		(property "Footprint" "Connector_PinSocket_2.54mm:PinSocket_1x02_P2.54mm_Vertical"
+		(property "Footprint" "Connector_PinHeader_1.27mm:PinHeader_1x02_P1.27mm_Vertical"
 			(at 93.98 62.23 0)
 			(effects
@@
 			)
 		)
-		(property "Footprint" "Resistor_SMD:R_0402_1005Metric"
+		(property "Footprint" "Resistor_SMD:R_0402_1005Metric_Pad0.72x0.64mm_HandSolder"
 			(at 111.76 29.718 90)
 			(effects
@@
 			)
 		)
-		(property "Footprint" "Capacitor_SMD:C_0603_1608Metric_Pad1.08x0.95mm_HandSolder"
+		(property "Footprint" "Capacitor_SMD:C_0402_1005Metric_Pad0.74x0.62mm_HandSolder"
 			(at 120.3452 76.2 0)
 			(effects
@@
 			)
 		)
-		(property "Footprint" "Connector_PinSocket_2.00mm:PinSocket_1x02_P2.00mm_Vertical"
+		(property "Footprint" "Connector_PinHeader_1.27mm:PinHeader_1x02_P1.27mm_Vertical"
 			(at 95.25 30.48 0)
 			(effects
@@
 			)
 		)
-		(property "Footprint" "Capacitor_SMD:C_0603_1608Metric_Pad1.08x0.95mm_HandSolder"
+		(property "Footprint" "Capacitor_SMD:C_0402_1005Metric_Pad0.74x0.62mm_HandSolder"
 			(at 120.3452 44.45 0)
 			(effects

Commit message: v0.9 draft routing was completed
Connections:
- net GND: now also J8.9 (Pin_9); no longer J8.10 (Pin_10)
- net K1: now also J8.2 (Pin_2); no longer J8.1 (Pin_1)
- net K2: now also J8.1 (Pin_1); no longer J8.2 (Pin_2)
- net K3: now also J8.4 (Pin_4); no longer J8.3 (Pin_3)
- net K4: now also J8.3 (Pin_3); no longer J8.4 (Pin_4)
- net K5: now also J8.6 (Pin_6); no longer J8.5 (Pin_5)
- net K6: now also J8.5 (Pin_5); no longer J8.6 (Pin_6)
- net K7: now also J8.8 (Pin_8); no longer J8.7 (Pin_7)
- net K8: now also J8.7 (Pin_7); no longer J8.8 (Pin_8)
- net K9: now also J8.10 (Pin_10); no longer J8.9 (Pin_9)
- net RX1+: now also X1.B10 (RX1-); no longer X1.B11 (RX1+)
- net RX1-: now also X1.B11 (RX1+); no longer X1.B10 (RX1-)
- net RX2+: now also X1.A11 (RX2+); no longer X1.A10 (RX2-)
- net RX2-: now also X1.A10 (RX2-); no longer X1.A11 (RX2+)
- net TX1+: now also X1.A2 (TX1+); no longer X1.A3 (TX1-)
- net TX1-: now also X1.A3 (TX1-); no longer X1.A2 (TX1+)
